Commit message: Task1 final

File: my_rb1_description/urdf/my_rb1_robot.urdf (robot description, URDF)
Before this commit: robot my_rb1_robot, 7 links, 6 joints
Links:
- link back_castor: geometry collision sphere radius=0.025; visual sphere radius=0.025
- link base_footprint: mass 20 -> 0.5
- link base_link: mass 20 -> 19
- link front_castor: geometry collision sphere radius=0.025; visual sphere radius=0.025
- link front_laser: mass 1 -> 0.5
- link left_wheel: geometry collision cylinder length=0.1 radius=0.025; visual cylinder length=0.1 radius=0.025
- link right_wheel: geometry collision cylinder length=0.1 radius=0.025; visual cylinder length=0.1 radius=0.025

Commit message: Task3

File: my_rb1_description/urdf/my_rb1_robot.urdf (robot description, URDF)
Before this commit: robot my_rb1_robot, 7 links, 6 joints
Joints:
- joint joint_base_back_castor: limit effort=10000 velocity=1000 -> effort=100 velocity=10
- joint joint_base_link_front_castor: limit effort=10000 velocity=1000 -> effort=100 velocity=10
- joint joint_base_link_front_laser: limit effort=10000 velocity=1000 -> effort=100 velocity=10
- joint joint_base_link_left_wheel: limit effort=10000 velocity=1000 -> effort=100 velocity=10
- joint joint_base_link_right_wheel: limit effort=10000 velocity=1000 -> effort=100 velocity=10

Commit message: Checkpoint 2

File: my_rb1_description/urdf/my_rb1_robot.urdf (robot description, URDF)
Before this commit: robot my_rb1_robot, 7 links, 6 joints
Links:
- link base_link: mass 19 -> 20.0
Joints:
- removed joint joint_base_back_castor
- added joint joint_base_link_back_castor: type fixed, parent base_link, child back_castor, origin xyz=-0.1 0 -0.15 rpy=0 0 0, axis 0 1 0, limit effort=100 velocity=10
- joint joint_base_footprint_base_link: limit (none) -> effort=10000 velocity=1000
- joint joint_base_link_front_laser: limit effort=100 velocity=10 -> effort=10000 velocity=1000
